File: hardware/EPM570_LinuxCNC.kicad_sch (KiCad schematic)
At the start: 56 parts, among them J1 PI Connector, J2 POWER +24V, J4 JTAG, J6 SERVO OUTPUTS, J7 SPI, J8 RS-485, U1 EPM570T100, U13 MAX3485, U2 74HCT244, U7 AMS1117-3.3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

Commit message: PCB fixes. Added pull down resistors.
Parts:
- added R128, R129, R130, R131, R132, R133: 50K, Resistor_SMD:R_0603_1608Metric, symbol Device:R
Connections:
- net DATA_ADDR: now also R131.1
- net DATA_READY: now also R130.1
- net DATA_RW: now also R129.1
- net GND: now also R128.2, R129.2, R130.2, R131.2, R132.2, R133.2
- net INPUT_INTERRUPT: now also R133.1
- net PULSE_BUFFER_EMPTY: now also R132.1
- net PULSE_BUFFER_LOCK: now also R128.1
Other:
- moved on the sheet: C11, C14, C15, D2, D35, D36, H1, H10, H2, H3, H4, H5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
